File: pcb/locket.kicad_sch (KiCad schematic)
At the start: 19 parts, among them J1 Conn_01x24_Pin, J2 USB_C_Receptacle_USB2.0_16P, SW1 SW_Push, U1 ESP32-S3-WROOM-1, U3 TLV73328PDBV, U5 MIC5356-SGYMME, U6 USBLC6-2SC6

Commit message: schematic final and starting layout
Parts:
- added BT1: Battery_Cell, Connector_JST:JST_XH_S2B-XH-A_1x02_P2.50mm_Horizontal, symbol Device:Battery_Cell
- added C2, C3, C8, C9: 2.2u, Capacitor_SMD:C_0805_2012Metric, symbol Device:C
- added J3: Conn_01x14_Pin, Connector_PinSocket_2.54mm:PinSocket_1x14_P2.54mm_Vertical, symbol Connector:Conn_01x14_Pin
- added L1: 2.2uH, Inductor_SMD:L_0805_2012Metric, symbol Device:L
- added Q1: AO8810, mykicadfootprints:TSSOP-8_L4.4-W3.0-P0.65-LS6.4-BL, symbol New_Library:AO8810
- added R1: 300, Resistor_SMD:R_0805_2012Metric, symbol Device:R
- added R2, R3: 5.1k, Resistor_SMD:R_0603_1608Metric, symbol Device:R
- added R4: 45k, Resistor_SMD:R_0805_2012Metric, symbol Device:R
- added U2: MCP73812T-420I-OT, Package_TO_SOT_SMD:SOT-23-5, symbol Battery_Management:MCP73812T-420I-OT
- added U3: BQ297xy, Package_SON:WSON-6_1.5x1.5mm_P0.5mm, symbol Battery_Management:BQ297xy
- added U5: TLV61070ADBV, Package_TO_SOT_SMD:SOT-23-6, symbol Regulator_Switching:TLV61070ADBV
- C1: renamed from C2; footprint (none) -> Capacitor_SMD:C_0805_2012Metric
- C10: renamed from C4; value 22u -> 10u; footprint (none) -> Capacitor_SMD:C_0805_2012Metric
- C11: renamed from C1; footprint (none) -> Capacitor_SMD:C_0805_2012Metric
- C4: renamed from C6; footprint (none) -> Capacitor_SMD:C_0805_2012Metric
- C5: value C -> 0.1u; footprint (none) -> Capacitor_SMD:C_0805_2012Metric
- C6: renamed from C7; footprint (none) -> Capacitor_SMD:C_0805_2012Metric
- C7: renamed from C8; footprint (none) -> Capacitor_SMD:C_0805_2012Metric
- J1: renamed from J2; footprint (none) -> Connector_USB:USB_C_Receptacle_HRO_TYPE-C-31-M-12
- J2: renamed from J1; footprint (none) -> mykicadfootprints:FPC-SMD_P0.50-24P_QCHF-SM-H2.0
- R5: footprint (none) -> Resistor_SMD:R_0603_1608Metric
- R6: renamed from R4; footprint (none) -> Resistor_SMD:R_0603_1608Metric
- R7: renamed from R3; footprint (none) -> Resistor_SMD:R_0603_1608Metric
- R8: renamed from R1; footprint (none) -> Resistor_SMD:R_0603_1608Metric
- R9: renamed from R2; footprint (none) -> Resistor_SMD:R_0603_1608Metric
- SW1: footprint (none) -> Button_Switch_THT:SW_Slide_SPDT_Straight_CK_OS102011MS2Q
- renumbered U3 to U1, U5 to U4, U1 to U7
Connections:
- net 1V8_EN is gone; now on net CAM_PWR_EN: U4.4 (EN2)
- net 2V8_EN is gone; now on net CAM_PWR_EN: U1.3 (EN)
- net +1V8: now also C1.1, U1.5 (OUT); no longer C6.1, U4.7 (VOUT2)
- net +2V8: now also C6.1, U4.7 (VOUT2); no longer C1.1, U1.5 (OUT)
- net +5V: now also C2.1, C9.1, J3.14 (Pin_14), R4.2, U2.1 (CE), U2.4 (V_{DD}), U5.5 (V_{OUT}); no longer C4.1, U4.1 (VIN), U4.5 (EN1)
- net DISP_BACKLIGHT: now also U7.32 (IO39), J3.7 (Pin_7); no longer U7.37 (TXD0)
- net DISP_CLK: now also U7.33 (IO40), J3.8 (Pin_8); no longer U7.35 (IO42)
- net DISP_CS: now also U7.37 (TXD0), J3.12 (Pin_12); no longer U7.31 (IO38)
- net DISP_DC: now also U7.35 (IO42), J3.10 (Pin_10); no longer U7.33 (IO40)
- net DISP_MISO: now also U7.31 (IO38), J3.6 (Pin_6); no longer U7.36 (RXD0)
- net DISP_MOSI: now also J3.9 (Pin_9)
- net DISP_RST: now also U7.36 (RXD0), J3.11 (Pin_11); no longer U7.32 (IO39)
- net GND: now also C2.2, C3.2, C8.2, C9.2, J3.13 (Pin_13), Q1.6 (S2), Q1.7 (S2), R2.1, R3.1, U2.2 (V_{SS}), U5.2 (GND)
- net TOUCH_CLK: now also U7.25 (IO48), J3.5 (Pin_5); no longer U7.24 (IO47)
- net TOUCH_INT: now also U7.22 (IO14), J3.2 (Pin_2); no longer U7.23 (IO21)
- net TOUCH_RST: now also U7.24 (IO47), J3.4 (Pin_4); no longer U7.22 (IO14)
- net TOUCH_SDA: now also U7.23 (IO21), J3.3 (Pin_3); no longer U7.25 (IO48)
- net USB_D-: now reaches U6.6 (I/O1), U7.13 (USB_D-)
- net USB_D+: now reaches U6.4 (I/O2), U7.14 (USB_D+)
- net CAM_PWR_EN: now reaches U7.15 (IO3)
- net at R5.2: now also R4.1, U5.4 (V_{FB}); no longer U7.16 (IO46)
- net DISP_PWR_EN: now reaches U7.26 (IO45)
- net DISP_PWR_EN: now also U5.3 (EN)
- net USBC_D+: now reaches J1.A6 (D+), J1.B6 (D+), U6.3 (I/O2)
- net USBC_D-: now reaches J1.A7 (D-), J1.B7 (D-), U6.1 (I/O1)
- net at C5.1: now also R1.1, U3.5 (BAT)
- net VBAT_SENSE: now reaches C5.2
- net VBAT_SENSE: now also BT1.2 (-), Q1.2 (S1), Q1.3 (S1), U3.4 (VSS)
- new net: R3.2, U2.5 (PROG)
- new net: Q1.5 (G2), U3.2 (Cout)
- new net: Q1.4 (G1), U3.3 (Dout)
- new net: L1.2, U5.1 (SW)
- new net LiPo+: BT1.1 (+), C3.1, C4.1, C8.1, L1.1, R1.2, U2.3 (V_{BAT}), U4.1 (VIN), U4.5 (EN1), U5.6 (V_{IN})
- new net SD_CS: J3.1 (Pin_1), U7.16 (IO46)
- new net VBAT_SENSE-: R2.2, U3.6 (V-)
- no-connect marks 4 -> 9
Other:
- note added: "500mA charge set"
- note added: "VREF = 500mV, VOUT = 5V R1 = (VOUT / VREF - 1) * R2 R1 = 9R2"
- note added: "max charge current we want to allow: 500mA voltage drop across FETs = 0.5 * Rdsson of FET Overcharge current threshold of BQ2970 is 100mV 100mV > 0.5A * Rdsson"
- title: (none) -> locket
- moved on the sheet: C10, C11, C4, C6, C7, J1, J2, R6, R7, R8, R9, SW1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
